Commit message: fixing python depednencies installed with pip

File: src/interfacing/eve_description/urdf/eve_mirror_mount_left.xacro (robot description, xacro)
@@ -1,26 +1,14 @@
 <?xml version="1.0"?>
 <robot xmlns:xacro="http://ros.org/wiki/xacro">
-  <!-- Simplified sensor mount with yaw calibration -->
-  <xacro:macro name="sensor_yaw_mount" params="name parent_link child_link x y z roll pitch yaw">
-    <joint name="${name}_yaw" type="revolute">
-      <parent link="${parent_link}"/>
-      <child link="${child_link}"/>
-      <origin xyz="${x} ${y} ${z}" rpy="${roll} ${pitch} ${yaw}"/>
-      <axis xyz="0 0 1"/>
-      <limit effort="0" velocity="0.01" lower="-0.2" upper="0.2"/>
-    </joint>
-  </xacro:macro>
-  <!-- Roof mount macro - allows parent specification -->
+  <!-- Mirror mount macro - allows parent specification -->
   <xacro:macro name="mirror_mount_left" params="parent *origin">
-    <!-- Roof mount for all sensors -->
+    <!-- Mirror mount for all sensors -->
     <link name="mirror_mount_left"/>
-    <joint name="mirror_mount_left_joint" type="revolute">
+    <joint name="mirror_mount_left_joint" type="fixed">
       <parent link="${parent}"/>
       <child link="mirror_mount_left"/>
       <xacro:insert_block name="origin"/>
-      <axis xyz="0 0 1"/>
-      <limit effort="0" velocity="0" lower="-0.0001" upper="0.0001"/>
     </joint>
-    <!-- Top LiDAR -->
+    <!-- Left LiDAR -->
     <link name="lidar_left">
       <visual>
@@ -40,6 +28,9 @@
       </collision>
     </link>
-    <xacro:sensor_yaw_mount name="lidar_left_mount" parent_link="mirror_mount_left" child_link="lidar_left"
-                            x="0" y="0" z="0" roll="0" pitch="0" yaw="0"/>
+    <joint name="lidar_left_mount_yaw" type="fixed">
+      <parent link="mirror_mount_left"/>
+      <child link="lidar_left"/>
+      <origin xyz="0 0 0" rpy="0 0 0"/>
+    </joint>
   </xacro:macro>
 </robot>

File: src/interfacing/eve_description/urdf/eve_mirror_mount_right.xacro (robot description, xacro)
@@ -1,26 +1,14 @@
 <?xml version="1.0"?>
 <robot xmlns:xacro="http://ros.org/wiki/xacro">
-  <!-- Simplified sensor mount with yaw calibration -->
-  <xacro:macro name="sensor_yaw_mount" params="name parent_link child_link x y z roll pitch yaw">
-    <joint name="${name}_yaw" type="revolute">
-      <parent link="${parent_link}"/>
-      <child link="${child_link}"/>
-      <origin xyz="${x} ${y} ${z}" rpy="${roll} ${pitch} ${yaw}"/>
-      <axis xyz="0 0 1"/>
-      <limit effort="0" velocity="0.01" lower="-0.2" upper="0.2"/>
-    </joint>
-  </xacro:macro>
-  <!-- Roof mount macro - allows parent specification -->
+  <!-- Mirror mount macro - allows parent specification -->
   <xacro:macro name="mirror_mount_right" params="parent *origin">
-    <!-- Roof mount for all sensors -->
+    <!-- Mirror mount for all sensors -->
     <link name="mirror_mount_right"/>
-    <joint name="mirror_mount_right_joint" type="revolute">
+    <joint name="mirror_mount_right_joint" type="fixed">
       <parent link="${parent}"/>
       <child link="mirror_mount_right"/>
       <xacro:insert_block name="origin"/>
-      <axis xyz="0 0 1"/>
-      <limit effort="0" velocity="0" lower="-0.0001" upper="0.0001"/>
     </joint>
-    <!-- Top LiDAR -->
+    <!-- Right LiDAR -->
     <link name="lidar_right">
       <visual>
@@ -40,6 +28,9 @@
       </collision>
     </link>
-    <xacro:sensor_yaw_mount name="lidar_right_mount" parent_link="mirror_mount_right" child_link="lidar_right"
-                            x="0" y="0" z="0" roll="0" pitch="0" yaw="0"/>
+    <joint name="lidar_right_mount_yaw" type="fixed">
+      <parent link="mirror_mount_right"/>
+      <child link="lidar_right"/>
+      <origin xyz="0 0 0" rpy="0 0 0"/>
+    </joint>
   </xacro:macro>
 </robot>

File: src/interfacing/eve_description/urdf/eve_roof_mount.xacro (robot description, xacro)
@@ -1,24 +1,12 @@
 <?xml version="1.0"?>
 <robot xmlns:xacro="http://ros.org/wiki/xacro">
-  <!-- Simplified sensor mount with yaw calibration -->
-  <xacro:macro name="sensor_yaw_mount" params="name parent_link child_link x y z roll pitch yaw">
-    <joint name="${name}_yaw" type="revolute">
-      <parent link="${parent_link}"/>
-      <child link="${child_link}"/>
-      <origin xyz="${x} ${y} ${z}" rpy="${roll} ${pitch} ${yaw}"/>
-      <axis xyz="0 0 1"/>
-      <limit effort="0" velocity="0.01" lower="-0.2" upper="0.2"/>
-    </joint>
-  </xacro:macro>
   <!-- Roof mount macro - allows parent specification -->
   <xacro:macro name="roof_mount" params="parent *origin">
     <!-- Roof mount for all sensors -->
     <link name="roof_mount"/>
-    <joint name="roof_mount_joint" type="revolute">
+    <joint name="roof_mount_joint" type="fixed">
       <parent link="${parent}"/>
       <child link="roof_mount"/>
       <xacro:insert_block name="origin"/>
-      <axis xyz="0 0 1"/>
-      <limit effort="0" velocity="0" lower="-0.0001" upper="0.0001"/>
     </joint>
     <!-- Top LiDAR -->
@@ -40,6 +28,9 @@
       </collision>
     </link>
-    <xacro:sensor_yaw_mount name="lidar_top_mount" parent_link="roof_mount" child_link="lidar_top"
-                            x="0" y="0" z="0.35" roll="0" pitch="0" yaw="0"/>
+    <joint name="lidar_top_mount_yaw" type="fixed">
+      <parent link="roof_mount"/>
+      <child link="lidar_top"/>
+      <origin xyz="0 0 0.35" rpy="0 0 0"/>
+    </joint>
     <!-- GPS/IMU Antenna -->
     <link name="gps_imu_antenna">
@@ -60,6 +51,9 @@
       </collision>
     </link>
-    <xacro:sensor_yaw_mount name="gps_imu_mount" parent_link="roof_mount" child_link="gps_imu_antenna"
-                            x="-0.5600" y="0" z="0" roll="0" pitch="0" yaw="0"/>
+    <joint name="gps_imu_mount_yaw" type="fixed">
+      <parent link="roof_mount"/>
+      <child link="gps_imu_antenna"/>
+      <origin xyz="-0.5600 0 0" rpy="0 0 0"/>
+    </joint>
     <!-- Roof-Mounted Cameras -->
     <link name="camera_front_center">
@@ -80,6 +74,9 @@
       </collision>
     </link>
-    <xacro:sensor_yaw_mount name="camera_front_center_mount" parent_link="roof_mount" child_link="camera_front_center"
-                            x="0.2375" y="0" z="0.185" roll="0" pitch="0" yaw="0"/>
+    <joint name="camera_front_center_mount_yaw" type="fixed">
+      <parent link="roof_mount"/>
+      <child link="camera_front_center"/>
+      <origin xyz="0.2375 0 0.185" rpy="0 0 0"/>
+    </joint>
     <link name="camera_front_left">
       <visual>
@@ -99,6 +96,9 @@
       </collision>
     </link>
-    <xacro:sensor_yaw_mount name="camera_front_left_mount" parent_link="roof_mount" child_link="camera_front_left"
-                            x="0.1875" y="0.185" z="0.185" roll="0" pitch="0" yaw="${pi/4}"/>
+    <joint name="camera_front_left_mount_yaw" type="fixed">
+      <parent link="roof_mount"/>
+      <child link="camera_front_left"/>
+      <origin xyz="0.1875 0.185 0.185" rpy="0 0 ${pi/4}"/>
+    </joint>
     <link name="camera_front_right">
       <visual>
@@ -118,6 +118,9 @@
       </collision>
     </link>
-    <xacro:sensor_yaw_mount name="camera_front_right_mount" parent_link="roof_mount" child_link="camera_front_right"
-                            x="0.1875" y="-0.185" z="0.185" roll="0" pitch="0" yaw="-${pi/4}"/>
+    <joint name="camera_front_right_mount_yaw" type="fixed">
+      <parent link="roof_mount"/>
+      <child link="camera_front_right"/>
+      <origin xyz="0.1875 -0.185 0.185" rpy="0 -0 -${pi/4}"/>
+    </joint>
   </xacro:macro>
 </robot>

Commit message: updating lidar extrinsic naming scheme

File: src/interfacing/eve_description/urdf/eve_mirror_mount_left.xacro (robot description, xacro)
@@ -11,5 +11,5 @@
     </joint>
     <!-- Left LiDAR -->
-    <link name="lidar_left">
+    <link name="lidar_NW">
       <visual>
         <origin xyz="0 0 0" rpy="0 0 0"/>
@@ -28,7 +28,7 @@
       </collision>
     </link>
-    <joint name="lidar_left_mount_yaw" type="fixed">
+    <joint name="lidar_NW_mount_yaw" type="fixed">
       <parent link="mirror_mount_left"/>
-      <child link="lidar_left"/>
+      <child link="lidar_NW"/>
       <origin xyz="0 0 0" rpy="0 0 0"/>
     </joint>

File: src/interfacing/eve_description/urdf/eve_mirror_mount_right.xacro (robot description, xacro)
@@ -11,5 +11,5 @@
     </joint>
     <!-- Right LiDAR -->
-    <link name="lidar_right">
+    <link name="lidar_NE">
       <visual>
         <origin xyz="0 0 0" rpy="0 0 0"/>
@@ -28,7 +28,7 @@
       </collision>
     </link>
-    <joint name="lidar_right_mount_yaw" type="fixed">
+    <joint name="lidar_NE_mount_yaw" type="fixed">
       <parent link="mirror_mount_right"/>
-      <child link="lidar_right"/>
+      <child link="lidar_NE"/>
       <origin xyz="0 0 0" rpy="0 0 0"/>
     </joint>
