Commit message: Eddy/update lidar extrinsic (#275)
* updating lidar extrinsic naming scheme

* naming convention and flip

* pre-commit

File: src/interfacing/eve_description/urdf/eve_mirror_mount_ne.xacro (robot description, xacro)
@@ -2,14 +2,14 @@
 <robot xmlns:xacro="http://ros.org/wiki/xacro">
   <!-- Mirror mount macro - allows parent specification -->
-  <xacro:macro name="mirror_mount_right" params="parent *origin">
+  <xacro:macro name="mirror_mount_nw" params="parent *origin">
     <!-- Mirror mount for all sensors -->
-    <link name="mirror_mount_right"/>
-    <joint name="mirror_mount_right_joint" type="fixed">
+    <link name="mirror_mount_nw"/>
+    <joint name="mirror_mount_nw_joint" type="fixed">
       <parent link="${parent}"/>
-      <child link="mirror_mount_right"/>
+      <child link="mirror_mount_nw"/>
       <xacro:insert_block name="origin"/>
     </joint>
-    <!-- Right LiDAR -->
-    <link name="lidar_right">
+    <!-- Left LiDAR -->
+    <link name="lidar_nw">
       <visual>
         <origin xyz="0 0 0" rpy="0 0 0"/>
@@ -28,7 +28,7 @@
       </collision>
     </link>
-    <joint name="lidar_right_mount_yaw" type="fixed">
-      <parent link="mirror_mount_right"/>
-      <child link="lidar_right"/>
+    <joint name="lidar_nw_mount_yaw" type="fixed">
+      <parent link="mirror_mount_nw"/>
+      <child link="lidar_nw"/>
       <origin xyz="0 0 0" rpy="0 0 0"/>
     </joint>

File: src/interfacing/eve_description/urdf/eve_mirror_mount_nw.xacro (robot description, xacro)
@@ -2,14 +2,14 @@
 <robot xmlns:xacro="http://ros.org/wiki/xacro">
   <!-- Mirror mount macro - allows parent specification -->
-  <xacro:macro name="mirror_mount_left" params="parent *origin">
+  <xacro:macro name="mirror_mount_ne" params="parent *origin">
     <!-- Mirror mount for all sensors -->
-    <link name="mirror_mount_left"/>
-    <joint name="mirror_mount_left_joint" type="fixed">
+    <link name="mirror_mount_ne"/>
+    <joint name="mirror_mount_ne_joint" type="fixed">
       <parent link="${parent}"/>
-      <child link="mirror_mount_left"/>
+      <child link="mirror_mount_ne"/>
       <xacro:insert_block name="origin"/>
     </joint>
-    <!-- Left LiDAR -->
-    <link name="lidar_left">
+    <!-- Right LiDAR -->
+    <link name="lidar_ne">
       <visual>
         <origin xyz="0 0 0" rpy="0 0 0"/>
@@ -28,7 +28,7 @@
       </collision>
     </link>
-    <joint name="lidar_left_mount_yaw" type="fixed">
-      <parent link="mirror_mount_left"/>
-      <child link="lidar_left"/>
+    <joint name="lidar_ne_mount_yaw" type="fixed">
+      <parent link="mirror_mount_ne"/>
+      <child link="lidar_ne"/>
       <origin xyz="0 0 0" rpy="0 0 0"/>
     </joint>
