Commit message: Update front 3 camera extrinsics

File: src/interfacing/eve_description/urdf/eve_roof_mount.xacro (robot description, xacro)
@@ -56,6 +56,8 @@
       <origin xyz="-0.5600 0 0" rpy="0 0 0"/>
     </joint>
+    <xacro:property name="camera_z" value="0.217"/>
+    <xacro:property name="pano_radius" value="0.240676"/>
     <!-- Roof-Mounted Cameras -->
-    <link name="camera_front_center">
+    <link name="camera_nn">
       <visual>
         <origin xyz="0 0 0" rpy="0 0 0"/>
@@ -74,10 +76,10 @@
       </collision>
     </link>
-    <joint name="camera_front_center_mount_yaw" type="fixed">
+    <joint name="camera_nn_mount_yaw" type="fixed">
       <parent link="roof_mount"/>
-      <child link="camera_front_center"/>
-      <origin xyz="0.2375 0 0.185" rpy="0 0 0"/>
+      <child link="camera_nn"/>
+      <origin xyz="${pano_radius} 0 ${camera_z}" rpy="0 0 0"/>
     </joint>
-    <link name="camera_front_left">
+    <link name="camera_pano_nw">
       <visual>
         <origin xyz="0 0 0" rpy="0 0 0"/>
@@ -96,10 +98,10 @@
       </collision>
     </link>
-    <joint name="camera_front_left_mount_yaw" type="fixed">
+    <joint name="camera_pano_nw_mount_yaw" type="fixed">
       <parent link="roof_mount"/>
-      <child link="camera_front_left"/>
-      <origin xyz="0.1875 0.185 0.185" rpy="0 0 ${pi/4}"/>
+      <child link="camera_pano_nw"/>
+      <origin xyz="${pano_radius/sqrt(2)} ${pano_radius/sqrt(2)} ${camera_z}" rpy="0 0 ${pi/4}"/>
     </joint>
-    <link name="camera_front_right">
+    <link name="camera_pano_ne">
       <visual>
         <origin xyz="0 0 0" rpy="0 0 0"/>
@@ -118,8 +120,8 @@
       </collision>
     </link>
-    <joint name="camera_front_right_mount_yaw" type="fixed">
+    <joint name="camera_pano_ne_mount_yaw" type="fixed">
       <parent link="roof_mount"/>
-      <child link="camera_front_right"/>
-      <origin xyz="0.1875 -0.185 0.185" rpy="0 -0 -${pi/4}"/>
+      <child link="camera_pano_ne"/>
+      <origin xyz="${pano_radius/sqrt(2)} -${pano_radius/sqrt(2)} ${camera_z}" rpy="0 -0 -${pi/4}"/>
     </joint>
   </xacro:macro>

Commit message: Add nominal extrinsics for all pano cameras

File: src/interfacing/eve_description/urdf/eve_roof_mount.xacro (robot description, xacro)
@@ -58,71 +58,41 @@
     <xacro:property name="camera_z" value="0.217"/>
     <xacro:property name="pano_radius" value="0.240676"/>
-    <!-- Roof-Mounted Cameras -->
-    <link name="camera_nn">
-      <visual>
-        <origin xyz="0 0 0" rpy="0 0 0"/>
-        <geometry>
-          <sphere radius="0.05"/>
-        </geometry>
-        <material name="red">
-          <color rgba="1.0 0.0 0.0 1"/>
-        </material>
-      </visual>
-      <collision>
-        <origin xyz="0 0 0" rpy="0 0 0"/>
-        <geometry>
-          <sphere radius="0.05"/>
-        </geometry>
-      </collision>
-    </link>
-    <joint name="camera_nn_mount_yaw" type="fixed">
-      <parent link="roof_mount"/>
-      <child link="camera_nn"/>
-      <origin xyz="${pano_radius} 0 ${camera_z}" rpy="0 0 0"/>
-    </joint>
-    <link name="camera_pano_nw">
-      <visual>
-        <origin xyz="0 0 0" rpy="0 0 0"/>
-        <geometry>
-          <sphere radius="0.05"/>
-        </geometry>
-        <material name="red">
-          <color rgba="1.0 0.0 0.0 1"/>
-        </material>
-      </visual>
-      <collision>
-        <origin xyz="0 0 0" rpy="0 0 0"/>
-        <geometry>
-          <sphere radius="0.05"/>
-        </geometry>
-      </collision>
-    </link>
-    <joint name="camera_pano_nw_mount_yaw" type="fixed">
-      <parent link="roof_mount"/>
-      <child link="camera_pano_nw"/>
-      <origin xyz="${pano_radius/sqrt(2)} ${pano_radius/sqrt(2)} ${camera_z}" rpy="0 0 ${pi/4}"/>
-    </joint>
-    <link name="camera_pano_ne">
-      <visual>
-        <origin xyz="0 0 0" rpy="0 0 0"/>
-        <geometry>
-          <sphere radius="0.05"/>
-        </geometry>
-        <material name="red">
-          <color rgba="1.0 0.0 0.0 1"/>
-        </material>
-      </visual>
-      <collision>
-        <origin xyz="0 0 0" rpy="0 0 0"/>
-        <geometry>
-          <sphere radius="0.05"/>
-        </geometry>
-      </collision>
-    </link>
-    <joint name="camera_pano_ne_mount_yaw" type="fixed">
-      <parent link="roof_mount"/>
-      <child link="camera_pano_ne"/>
-      <origin xyz="${pano_radius/sqrt(2)} -${pano_radius/sqrt(2)} ${camera_z}" rpy="0 -0 -${pi/4}"/>
-    </joint>
+    <xacro:property name="pano_cameras" value="8"/>
+    <xacro:property name="angle_increment" value="${2*pi/pano_cameras}"/>
+    <xacro:macro name="create_camera" params="index name">
+      <xacro:property name="angle" value="${-pi/4 - index * angle_increment}"/>
+      <xacro:property name="cam_x" value="${pano_radius * cos(angle)}"/>
+      <xacro:property name="cam_y" value="${pano_radius * sin(angle)}"/>
+      <link name="camera_pano_${name}">
+        <visual>
+          <origin xyz="0 0 0" rpy="0 0 0"/>
+          <geometry>
+            <sphere radius="0.05"/>
+          </geometry>
+          <material name="red">
+            <color rgba="1.0 0.0 0.0 1"/>
+          </material>
+        </visual>
+        <collision>
+          <origin xyz="0 0 0" rpy="0 0 0"/>
+          <geometry>
+            <sphere radius="0.05"/>
+          </geometry>
+        </collision>
+      </link>
+      <joint name="camera_pano_${name}_mount" type="fixed">
+        <parent link="roof_mount"/>
+        <child link="camera_pano_${name}"/>
+        <origin xyz="${cam_x} ${cam_y} ${camera_z}" rpy="0 0 ${angle}"/>
+      </joint>
+    </xacro:macro>
+    <xacro:create_camera index="0" name="ne"/>
+    <xacro:create_camera index="1" name="ee"/>
+    <xacro:create_camera index="2" name="se"/>
+    <xacro:create_camera index="3" name="ss"/>
+    <xacro:create_camera index="4" name="sw"/>
+    <xacro:create_camera index="5" name="ww"/>
+    <xacro:create_camera index="6" name="nw"/>
+    <xacro:create_camera index="7" name="nn"/>
   </xacro:macro>
 </robot>

Commit message: Change coordinate frames for cameras to be RDF

File: src/interfacing/eve_description/urdf/eve_roof_mount.xacro (robot description, xacro)
@@ -66,5 +66,5 @@
       <link name="camera_pano_${name}">
         <visual>
-          <origin xyz="0 0 0" rpy="0 0 0"/>
+          <origin xyz="0 0 0" rpy="${-pi/2.0} 0 ${-pi/2.0}"/>
           <geometry>
             <sphere radius="0.05"/>
@@ -75,5 +75,5 @@
         </visual>
         <collision>
-          <origin xyz="0 0 0" rpy="0 0 0"/>
+          <origin xyz="0 0 0" rpy="${-pi/2.0} 0 ${-pi/2.0}"/>
           <geometry>
             <sphere radius="0.05"/>
@@ -81,8 +81,9 @@
         </collision>
       </link>
+      <!-- the additional rotation of -pi/2 is to go from FLU to RDF coordinate systems -->
       <joint name="camera_pano_${name}_mount" type="fixed">
         <parent link="roof_mount"/>
         <child link="camera_pano_${name}"/>
-        <origin xyz="${cam_x} ${cam_y} ${camera_z}" rpy="0 0 ${angle}"/>
+        <origin xyz="${cam_x} ${cam_y} ${camera_z}" rpy="${-pi/2} 0 ${angle - pi/2}"/>
       </joint>
     </xacro:macro>

Commit message: Calibrate panorama intrinsics and add nominal extrinsics (#269)

File: src/interfacing/eve_description/urdf/eve_roof_mount.xacro (robot description, xacro)
@@ -56,71 +56,44 @@
       <origin xyz="-0.5600 0 0" rpy="0 0 0"/>
     </joint>
-    <!-- Roof-Mounted Cameras -->
-    <link name="camera_front_center">
-      <visual>
-        <origin xyz="0 0 0" rpy="0 0 0"/>
-        <geometry>
-          <sphere radius="0.05"/>
-        </geometry>
-        <material name="red">
-          <color rgba="1.0 0.0 0.0 1"/>
-        </material>
-      </visual>
-      <collision>
-        <origin xyz="0 0 0" rpy="0 0 0"/>
-        <geometry>
-          <sphere radius="0.05"/>
-        </geometry>
-      </collision>
-    </link>
-    <joint name="camera_front_center_mount_yaw" type="fixed">
-      <parent link="roof_mount"/>
-      <child link="camera_front_center"/>
-      <origin xyz="0.2375 0 0.185" rpy="0 0 0"/>
-    </joint>
-    <link name="camera_front_left">
-      <visual>
-        <origin xyz="0 0 0" rpy="0 0 0"/>
-        <geometry>
-          <sphere radius="0.05"/>
-        </geometry>
-        <material name="red">
-          <color rgba="1.0 0.0 0.0 1"/>
-        </material>
-      </visual>
-      <collision>
-        <origin xyz="0 0 0" rpy="0 0 0"/>
-        <geometry>
-          <sphere radius="0.05"/>
-        </geometry>
-      </collision>
-    </link>
-    <joint name="camera_front_left_mount_yaw" type="fixed">
-      <parent link="roof_mount"/>
-      <child link="camera_front_left"/>
-      <origin xyz="0.1875 0.185 0.185" rpy="0 0 ${pi/4}"/>
-    </joint>
-    <link name="camera_front_right">
-      <visual>
-        <origin xyz="0 0 0" rpy="0 0 0"/>
-        <geometry>
-          <sphere radius="0.05"/>
-        </geometry>
-        <material name="red">
-          <color rgba="1.0 0.0 0.0 1"/>
-        </material>
-      </visual>
-      <collision>
-        <origin xyz="0 0 0" rpy="0 0 0"/>
-        <geometry>
-          <sphere radius="0.05"/>
-        </geometry>
-      </collision>
-    </link>
-    <joint name="camera_front_right_mount_yaw" type="fixed">
-      <parent link="roof_mount"/>
-      <child link="camera_front_right"/>
-      <origin xyz="0.1875 -0.185 0.185" rpy="0 -0 -${pi/4}"/>
-    </joint>
+    <xacro:property name="camera_z" value="0.217"/>
+    <xacro:property name="pano_radius" value="0.240676"/>
+    <xacro:property name="pano_cameras" value="8"/>
+    <xacro:property name="angle_increment" value="${2*pi/pano_cameras}"/>
+    <xacro:macro name="create_camera" params="index name">
+      <xacro:property name="angle" value="${-pi/4 - index * angle_increment}"/>
+      <xacro:property name="cam_x" value="${pano_radius * cos(angle)}"/>
+      <xacro:property name="cam_y" value="${pano_radius * sin(angle)}"/>
+      <link name="camera_pano_${name}">
+        <visual>
+          <origin xyz="0 0 0" rpy="${-pi/2.0} 0 ${-pi/2.0}"/>
+          <geometry>
+            <sphere radius="0.05"/>
+          </geometry>
+          <material name="red">
+            <color rgba="1.0 0.0 0.0 1"/>
+          </material>
+        </visual>
+        <collision>
+          <origin xyz="0 0 0" rpy="${-pi/2.0} 0 ${-pi/2.0}"/>
+          <geometry>
+            <sphere radius="0.05"/>
+          </geometry>
+        </collision>
+      </link>
+      <!-- the additional rotation of -pi/2 is to go from FLU to RDF coordinate systems -->
+      <joint name="camera_pano_${name}_mount" type="fixed">
+        <parent link="roof_mount"/>
+        <child link="camera_pano_${name}"/>
+        <origin xyz="${cam_x} ${cam_y} ${camera_z}" rpy="${-pi/2} 0 ${angle - pi/2}"/>
+      </joint>
+    </xacro:macro>
+    <xacro:create_camera index="0" name="ne"/>
+    <xacro:create_camera index="1" name="ee"/>
+    <xacro:create_camera index="2" name="se"/>
+    <xacro:create_camera index="3" name="ss"/>
+    <xacro:create_camera index="4" name="sw"/>
+    <xacro:create_camera index="5" name="ww"/>
+    <xacro:create_camera index="6" name="nw"/>
+    <xacro:create_camera index="7" name="nn"/>
   </xacro:macro>
 </robot>

Commit message: fixed yaw of lower cameras

File: src/interfacing/eve_description/urdf/eve_roof_mount.xacro (robot description, xacro)
@@ -99,39 +99,35 @@
   <!-- Lower cameras (nominal extrinsics; update xyz/rpy once measured) -->
   <xacro:macro name="lower_cameras" params="parent">
-    <!--
-      Convention: camera link is used directly as frame_id (no separate optical frame).
-      The additional roll of -pi/2 follows the pano camera convention to go from FLU to RDF.
-    -->
     <xacro:property name="low_cam_x" value="1.50"/>
     <xacro:property name="low_cam_y" value="0.85"/>
     <xacro:property name="low_cam_z" value="0.75"/>
-    <!-- Cardinal-ish yaws for nominal mounting directions -->
-    <xacro:property name="yaw_ne" value="${pi/4}"/>
-    <xacro:property name="yaw_se" value="${-pi/4}"/>
-    <xacro:property name="yaw_sw" value="${-3*pi/4}"/>
-    <xacro:property name="yaw_nw" value="${3*pi/4}"/>
-    <link name="camera_low_ne"/>
-    <joint name="camera_low_ne_mount" type="fixed">
+    <!-- Nominal yaws in the vehicle FLU frame (front=+x, left=+y), estimated from sensor_convention -->
+    <xacro:property name="yaw_ne" value="${-5*pi/6}"/>  <!-- ~ -150 deg -->
+    <xacro:property name="yaw_se" value="${-pi/6}"/>    <!-- ~ -30 deg -->
+    <xacro:property name="yaw_sw" value="${pi/6}"/>     <!-- ~ 30 deg -->
+    <xacro:property name="yaw_nw" value="${5*pi/6}"/>   <!-- ~ 150 deg -->
+    <link name="camera_lower_ne"/>
+    <joint name="camera_lower_ne_mount" type="fixed">
       <parent link="${parent}"/>
-      <child link="camera_low_ne"/>
+      <child link="camera_lower_ne"/>
       <origin xyz="${low_cam_x} ${-low_cam_y} ${low_cam_z}" rpy="${-pi/2} 0 ${yaw_ne - pi/2}"/>
     </joint>
-    <link name="camera_low_se"/>
-    <joint name="camera_low_se_mount" type="fixed">
+    <link name="camera_lower_se"/>
+    <joint name="camera_lower_se_mount" type="fixed">
       <parent link="${parent}"/>
-      <child link="camera_low_se"/>
-      <origin xyz="${low_cam_x} ${-low_cam_y} ${low_cam_z}" rpy="${-pi/2} 0 ${yaw_se - pi/2}"/>
+      <child link="camera_lower_se"/>
+      <origin xyz="${-low_cam_x} ${-low_cam_y} ${low_cam_z}" rpy="${-pi/2} 0 ${yaw_se - pi/2}"/>
     </joint>
-    <link name="camera_low_sw"/>
-    <joint name="camera_low_sw_mount" type="fixed">
+    <link name="camera_lower_sw"/>
+    <joint name="camera_lower_sw_mount" type="fixed">
       <parent link="${parent}"/>
-      <child link="camera_low_sw"/>
-      <origin xyz="${-low_cam_x} ${-low_cam_y} ${low_cam_z}" rpy="${-pi/2} 0 ${yaw_sw - pi/2}"/>
+      <child link="camera_lower_sw"/>
+      <origin xyz="${-low_cam_x} ${low_cam_y} ${low_cam_z}" rpy="${-pi/2} 0 ${yaw_sw - pi/2}"/>
     </joint>
-    <link name="camera_low_nw"/>
-    <joint name="camera_low_nw_mount" type="fixed">
+    <link name="camera_lower_nw"/>
+    <joint name="camera_lower_nw_mount" type="fixed">
       <parent link="${parent}"/>
-      <child link="camera_low_nw"/>
-      <origin xyz="${-low_cam_x} ${low_cam_y} ${low_cam_z}" rpy="${-pi/2} 0 ${yaw_nw - pi/2}"/>
+      <child link="camera_lower_nw"/>
+      <origin xyz="${low_cam_x} ${low_cam_y} ${low_cam_z}" rpy="${-pi/2} 0 ${yaw_nw - pi/2}"/>
     </joint>
   </xacro:macro>

Commit message: Update nominal extrinsics of lower camera

File: src/interfacing/eve_description/urdf/eve_roof_mount.xacro (robot description, xacro)
@@ -99,17 +99,18 @@
   <!-- Lower cameras (nominal extrinsics; update xyz/rpy once measured) -->
   <xacro:macro name="lower_cameras" params="parent">
-    <xacro:property name="low_cam_x" value="1.50"/>
-    <xacro:property name="low_cam_y" value="0.85"/>
-    <xacro:property name="low_cam_z" value="0.75"/>
+    <xacro:property name="low_cam_x_forward" value="0.6125"/>
+    <xacro:property name="low_cam_x_backward" value="0.775"/>
+    <xacro:property name="low_cam_y" value="0.725"/>
+    <xacro:property name="low_cam_z" value="0.034"/>
     <!-- Nominal yaws in the vehicle FLU frame (front=+x, left=+y), estimated from sensor_convention -->
-    <xacro:property name="yaw_ne" value="${-5*pi/6}"/>  <!-- ~ -150 deg -->
-    <xacro:property name="yaw_se" value="${-pi/6}"/>    <!-- ~ -30 deg -->
-    <xacro:property name="yaw_sw" value="${pi/6}"/>     <!-- ~ 30 deg -->
-    <xacro:property name="yaw_nw" value="${5*pi/6}"/>   <!-- ~ 150 deg -->
+    <xacro:property name="yaw_ne" value="${-2.4434}"/>  <!-- ~ -150 deg -->
+    <xacro:property name="yaw_se" value="${0.8726}"/>    <!-- ~ -30 deg -->
+    <xacro:property name="yaw_sw" value="${2.4434}"/>     <!-- ~ 30 deg -->
+    <xacro:property name="yaw_nw" value="${-0.8726}"/>   <!-- ~ 150 deg -->
     <link name="camera_lower_ne"/>
     <joint name="camera_lower_ne_mount" type="fixed">
       <parent link="${parent}"/>
       <child link="camera_lower_ne"/>
-      <origin xyz="${low_cam_x} ${-low_cam_y} ${low_cam_z}" rpy="${-pi/2} 0 ${yaw_ne - pi/2}"/>
+      <origin xyz="${low_cam_x_forward} ${-low_cam_y} ${-low_cam_z}" rpy="${-pi/2} 0 ${yaw_ne - pi/2}"/>
     </joint>
     <link name="camera_lower_se"/>
@@ -117,5 +118,5 @@
       <parent link="${parent}"/>
       <child link="camera_lower_se"/>
-      <origin xyz="${-low_cam_x} ${-low_cam_y} ${low_cam_z}" rpy="${-pi/2} 0 ${yaw_se - pi/2}"/>
+      <origin xyz="${-low_cam_x_backward} ${-low_cam_y} ${-low_cam_z}" rpy="${-pi/2} 0 ${yaw_se - pi}"/>
     </joint>
     <link name="camera_lower_sw"/>
@@ -123,5 +124,5 @@
       <parent link="${parent}"/>
       <child link="camera_lower_sw"/>
-      <origin xyz="${-low_cam_x} ${low_cam_y} ${low_cam_z}" rpy="${-pi/2} 0 ${yaw_sw - pi/2}"/>
+      <origin xyz="${-low_cam_x_backward} ${low_cam_y} ${-low_cam_z}" rpy="${-pi/2} 0 ${yaw_sw - pi}"/>
     </joint>
     <link name="camera_lower_nw"/>
@@ -129,5 +130,5 @@
       <parent link="${parent}"/>
       <child link="camera_lower_nw"/>
-      <origin xyz="${low_cam_x} ${low_cam_y} ${low_cam_z}" rpy="${-pi/2} 0 ${yaw_nw - pi/2}"/>
+      <origin xyz="${low_cam_x_forward} ${low_cam_y} ${-low_cam_z}" rpy="${-pi/2} 0 ${yaw_nw + pi/2}"/>
     </joint>
   </xacro:macro>

Commit message: imu_link

File: src/interfacing/eve_description/urdf/eve_roof_mount.xacro (robot description, xacro)
@@ -2,5 +2,5 @@
 <robot xmlns:xacro="http://ros.org/wiki/xacro">
   <!-- Roof mount macro - attaches sensors to the provided parent link -->
-  <xacro:macro name="roof_mount" params="parent">
+  <xacro:macro name="roof_mount" params="parent imu_xyz:='-0.5600 0 0' imu_rpy:='0 0 0'">
     <!-- Top LiDAR -->
     <link name="lidar_cc">
@@ -48,4 +48,26 @@
       <child link="gps_imu_antenna"/>
       <origin xyz="-0.5600 0 0" rpy="0 0 0"/>
+    </joint>
+    <link name="imu_link">
+      <visual>
+        <origin xyz="0 0 0" rpy="0 0 0"/>
+        <geometry>
+          <sphere radius="0.04"/>
+        </geometry>
+        <material name="green">
+          <color rgba="0.0 1.0 0.0 1"/>
+        </material>
+      </visual>
+      <collision>
+        <origin xyz="0 0 0" rpy="0 0 0"/>
+        <geometry>
+          <sphere radius="0.04"/>
+        </geometry>
+      </collision>
+    </link>
+    <joint name="imu_mount" type="fixed">
+      <parent link="${parent}"/>
+      <child link="imu_link"/>
+      <origin xyz="${imu_xyz}" rpy="${imu_rpy}"/>
     </joint>
     <xacro:property name="camera_z" value="0.217"/>

Commit message: add lidar_top to match the bag's topic name

File: src/interfacing/eve_description/urdf/eve_roof_mount.xacro (robot description, xacro)
@@ -25,4 +25,11 @@
       <child link="lidar_cc"/>
       <origin xyz="0 0 0.35" rpy="0 0 0"/>
+    </joint>
+    <!-- Alias frame to match bag/driver frame_id (lidar_top) -->
+    <link name="lidar_top"/>
+    <joint name="lidar_top_alias" type="fixed">
+      <parent link="lidar_cc"/>
+      <child link="lidar_top"/>
+      <origin xyz="0 0 0" rpy="0 0 0"/>
     </joint>
     <!-- GPS/IMU Antenna -->

Commit message: recording session mar 1

File: src/interfacing/eve_description/urdf/eve_roof_mount.xacro (robot description, xacro)
@@ -2,5 +2,5 @@
 <robot xmlns:xacro="http://ros.org/wiki/xacro">
   <!-- Roof mount macro - attaches sensors to the provided parent link -->
-  <xacro:macro name="roof_mount" params="parent">
+  <xacro:macro name="roof_mount" params="parent imu_xyz:='-0.5600 0 0' imu_rpy:='0 0 0'">
     <!-- Top LiDAR -->
     <link name="lidar_cc">
@@ -48,4 +48,26 @@
       <child link="gps_imu_antenna"/>
       <origin xyz="-0.5600 0 0" rpy="0 0 0"/>
+    </joint>
+    <link name="imu_link">
+      <visual>
+        <origin xyz="0 0 0" rpy="0 0 0"/>
+        <geometry>
+          <sphere radius="0.04"/>
+        </geometry>
+        <material name="green">
+          <color rgba="0.0 1.0 0.0 1"/>
+        </material>
+      </visual>
+      <collision>
+        <origin xyz="0 0 0" rpy="0 0 0"/>
+        <geometry>
+          <sphere radius="0.04"/>
+        </geometry>
+      </collision>
+    </link>
+    <joint name="imu_mount" type="fixed">
+      <parent link="lidar_cc"/>
+      <child link="imu_link"/>
+      <origin xyz="${imu_xyz}" rpy="${imu_rpy}"/>
     </joint>
     <xacro:property name="camera_z" value="0.217"/>
