Commit message: updated tf

File: src/interfacing/eve_description/urdf/eve_kia_soul_ev.xacro (robot description, xacro)
@@ -1,225 +1,17 @@
 <?xml version="1.0"?>
 <robot name="eve_kia_soul_ev" xmlns:xacro="http://ros.org/wiki/xacro">
-  <!-- Properties -->
-  <xacro:property name="length" value="4.14"/>
-  <xacro:property name="width" value="1.80"/>
-  <xacro:property name="height" value="1.60"/>
-  <xacro:property name="wheel_radius" value="0.3"/>
-  <xacro:property name="wheel_width" value="0.2"/>
-  <xacro:property name="wheelbase" value="2.51"/>
-  <xacro:property name="track_width" value="1.52"/>
-  <link name="base_link">
-    <visual>
-      <origin xyz="${wheelbase/2} 0 ${height/2}" rpy="0 0 0"/>
-      <geometry>
-        <box size="${length} ${width} ${height}"/>
-      </geometry>
-      <material name="grey">
-        <color rgba="0.5 0.5 0.5 1"/>
-      </material>
-    </visual>
-  </link>
-  <xacro:macro name="wheel" params="name x y z">
-    <link name="${name}_wheel">
-      <visual>
-        <origin xyz="0 0 0" rpy="0 0 0"/>
-        <geometry>
-          <cylinder radius="${wheel_radius}" length="${wheel_width}"/>
-        </geometry>
-        <material name="black">
-          <color rgba="0.0 0.0 0.0 1"/>
-        </material>
-      </visual>
-      <collision>
-        <origin xyz="0 0 0" rpy="0 0 0"/>
-        <geometry>
-          <cylinder radius="${wheel_radius}" length="${wheel_width}"/>
-        </geometry>
-      </collision>
-    </link>
-    <joint name="${name}_joint" type="continuous">
-      <parent link="base_link"/>
-      <child link="${name}_wheel"/>
-      <origin xyz="${x} ${y} ${z}" rpy="0 0 0"/>
-      <axis xyz="0 1 0"/>
-    </joint>
-  </xacro:macro>
-  <xacro:macro name="steering_wheel" params="name x y z">
-    <link name="${name}_knuckle"/>
-    <joint name="${name}_steering_joint" type="revolute">
-      <parent link="base_link"/>
-      <child link="${name}_knuckle"/>
-      <origin xyz="${x} ${y} ${z}" rpy="0 0 0"/>
-      <axis xyz="0 0 1"/>
-      <limit effort="10" velocity="1" lower="-0.785" upper="0.785"/> <!-- +/-45 deg -->
-    </joint>
-    <link name="${name}_wheel">
-      <visual>
-        <origin xyz="0 0 0" rpy="0 0 0"/>
-        <geometry>
-          <cylinder radius="${wheel_radius}" length="${wheel_width}"/>
-        </geometry>
-        <material name="black">
-          <color rgba="0.0 0.0 0.0 1"/>
-        </material>
-      </visual>
-      <collision>
-        <origin xyz="0 0 0" rpy="0 0 0"/>
-        <geometry>
-          <cylinder radius="${wheel_radius}" length="${wheel_width}"/>
-        </geometry>
-      </collision>
-    </link>
-    <joint name="${name}_wheel_joint" type="continuous">
-      <parent link="${name}_knuckle"/>
-      <child link="${name}_wheel"/>
-      <origin xyz="0 0 0" rpy="0 0 0"/>
-      <axis xyz="0 1 0"/>
-    </joint>
-  </xacro:macro>
-  <!-- 6-DOF sensor mount for online calibration -->
-  <!-- Uses chain of joints instead of floating joint (floating not supported by robot_state_publisher) -->
-  <xacro:macro name="sensor_6dof_mount" params="name parent_link child_link x y z roll pitch yaw">
-    <!-- Translation stages -->
-    <link name="${name}_x_translation"/>
-    <joint name="${name}_x" type="prismatic">
-      <parent link="${parent_link}"/>
-      <child link="${name}_x_translation"/>
-      <origin xyz="${x} ${y} ${z}" rpy="0 0 0"/>
-      <axis xyz="1 0 0"/>
-      <limit effort="0" velocity="0.01" lower="-0.1" upper="0.1"/>
-    </joint>
-    <link name="${name}_y_translation"/>
-    <joint name="${name}_y" type="prismatic">
-      <parent link="${name}_x_translation"/>
-      <child link="${name}_y_translation"/>
-      <origin xyz="0 0 0" rpy="0 0 0"/>
-      <axis xyz="0 1 0"/>
-      <limit effort="0" velocity="0.01" lower="-0.1" upper="0.1"/>
-    </joint>
-    <link name="${name}_z_translation"/>
-    <joint name="${name}_z" type="prismatic">
-      <parent link="${name}_y_translation"/>
-      <child link="${name}_z_translation"/>
-      <origin xyz="0 0 0" rpy="0 0 0"/>
-      <axis xyz="0 0 1"/>
-      <limit effort="0" velocity="0.01" lower="-0.1" upper="0.1"/>
-    </joint>
-    <!-- Rotation stages -->
-    <link name="${name}_roll_rotation"/>
-    <joint name="${name}_roll" type="revolute">
-      <parent link="${name}_z_translation"/>
-      <child link="${name}_roll_rotation"/>
-      <origin xyz="0 0 0" rpy="${roll} 0 0"/>
-      <axis xyz="1 0 0"/>
-      <limit effort="0" velocity="0.01" lower="-0.1" upper="0.1"/>
-    </joint>
-    <link name="${name}_pitch_rotation"/>
-    <joint name="${name}_pitch" type="revolute">
-      <parent link="${name}_roll_rotation"/>
-      <child link="${name}_pitch_rotation"/>
-      <origin xyz="0 0 0" rpy="0 ${pitch} 0"/>
-      <axis xyz="0 1 0"/>
-      <limit effort="0" velocity="0.01" lower="-0.1" upper="0.1"/>
-    </joint>
-    <link name="${name}_yaw_rotation"/>
-    <joint name="${name}_yaw" type="revolute">
-      <parent link="${name}_pitch_rotation"/>
-      <child link="${name}_yaw_rotation"/>
-      <origin xyz="0 0 0" rpy="0 0 ${yaw}"/>
-      <axis xyz="0 0 1"/>
-      <limit effort="0" velocity="0.01" lower="-0.1" upper="0.1"/>
-    </joint>
-    <!-- Final connection to sensor -->
-    <joint name="${name}_fixed" type="fixed">
-      <parent link="${name}_yaw_rotation"/>
-      <child link="${child_link}"/>
-      <origin xyz="0 0 0" rpy="0 0 0"/>
-    </joint>
-  </xacro:macro>
-  <!-- Rear Wheels -->
-  <xacro:wheel name="rear_left" x="0" y="${track_width/2}" z="${wheel_radius}"/>
-  <xacro:wheel name="rear_right" x="0" y="-${track_width/2}" z="${wheel_radius}"/>
-  <!-- Front Wheels with Steering -->
-  <xacro:steering_wheel name="front_left" x="${wheelbase}" y="${track_width/2}" z="${wheel_radius}"/>
-  <xacro:steering_wheel name="front_right" x="${wheelbase}" y="-${track_width/2}" z="${wheel_radius}"/>
-<link name="lidar_top">
-  <visual>
-    <origin xyz="0 0 0" rpy="0 0 0"/>
-    <geometry>
-      <cylinder radius="0.1" length="0.15"/>
-    </geometry>
-    <material name="black">
-      <color rgba="0 0 0 1"/>
-    </material>
-  </visual>
-  <collision>
-    <origin xyz="0 0 0" rpy="0 0 0"/>
-    <geometry>
-      <cylinder radius="0.1" length="0.15"/>
-    </geometry>
-  </collision>
-</link>
-<xacro:sensor_6dof_mount name="lidar_top_mount" parent_link="base_link" child_link="lidar_top"
-                          x="-0.55" y="0" z="2.07" roll="0" pitch="0" yaw="0"/>
-<!-- Left Mirror LiDAR -->
-<link name="lidar_left">
-  <visual>
-    <origin xyz="0 0 0" rpy="0 0 0"/>
-    <geometry>
-      <cylinder radius="0.08" length="0.12"/>
-    </geometry>
-    <material name="black">
-      <color rgba="0 0 0 1"/>
-    </material>
-  </visual>
-  <collision>
-    <origin xyz="0 0 0" rpy="0 0 0"/>
-    <geometry>
-      <cylinder radius="0.08" length="0.12"/>
-    </geometry>
-  </collision>
-</link>
-<xacro:sensor_6dof_mount name="lidar_left_mount" parent_link="base_link" child_link="lidar_left"
-                          x="-0.55" y="1" z="2.07" roll="0" pitch="0" yaw="2"/>
-<!-- Right Mirror LiDAR -->
-<link name="lidar_right">
-  <visual>
-    <origin xyz="0 0 0" rpy="0 0 0"/>
-    <geometry>
-      <cylinder radius="0.08" length="0.12"/>
-    </geometry>
-    <material name="black">
-      <color rgba="0 0 0 1"/>
-    </material>
-  </visual>
-  <collision>
-    <origin xyz="0 0 0" rpy="0 0 0"/>
-    <geometry>
-      <cylinder radius="0.08" length="0.12"/>
-    </geometry>
-  </collision>
-</link>
-<xacro:sensor_6dof_mount name="lidar_right_mount" parent_link="base_link" child_link="lidar_right"
-                          x="-0.55" y="-1" z="2.07" roll="0" pitch="0" yaw="2"/>
-<!-- GPS/IMU Antenna -->
-<link name="gps_imu_antenna">
-  <visual>
-    <origin xyz="0 0 0" rpy="0 0 0"/>
-    <geometry>
-      <sphere radius="0.05"/>
-    </geometry>
-    <material name="blue">
-      <color rgba="0.0 0.0 1.0 1"/>
-    </material>
-  </visual>
-  <collision>
-    <origin xyz="0 0 0" rpy="0 0 0"/>
-    <geometry>
-      <sphere radius="0.05"/>
-    </geometry>
-  </collision>
-</link>
-<xacro:sensor_6dof_mount name="gps_imu_mount" parent_link="base_link" child_link="gps_imu_antenna"
-                          x="-1.0326" y="0" z="1.689" roll="0" pitch="0" yaw="0"/>
+  <!-- Base link (root of the robot) -->
+  <link name="base_link"/>
+  <!-- Include chassis -->
+  <xacro:include filename="eve_chassis.xacro"/>
+  <!-- Instantiate chassis with position relative to base_link -->
+  <xacro:chassis parent="base_link">
+    <origin xyz="-0.8629 0 0" rpy="0 0 0"/>
+  </xacro:chassis>
+  <!-- Include roof mount and sensors -->
+  <xacro:include filename="eve_roof_mount.xacro"/>
+  <!-- Instantiate roof mount with position relative to chassis -->
+  <xacro:roof_mount parent="base_link">
+    <origin xyz="0 0 1.76" rpy="0 0 0"/>
+  </xacro:roof_mount>
 </robot>

Commit message: tested three lidar launch

File: src/interfacing/eve_description/urdf/eve_kia_soul_ev.xacro (robot description, xacro)
@@ -15,3 +15,12 @@
     <origin xyz="0 0 1.76" rpy="0 0 0"/>
   </xacro:roof_mount>
+  <!-- Include mirror mounts and sensors -->
+  <xacro:include filename="eve_mirror_mount_left.xacro"/>
+  <xacro:include filename="eve_mirror_mount_right.xacro"/>
+  <xacro:mirror_mount_left parent="base_link">
+    <origin xyz="0.95 0.88 1.26" rpy="0 0 0"/>
+  </xacro:mirror_mount_left>
+  <xacro:mirror_mount_right parent="base_link">
+    <origin xyz="0.95 -0.88 1.26" rpy="0 0 0"/>
+  </xacro:mirror_mount_right>
 </robot>

Commit message: cleaning up PR

File: src/interfacing/eve_description/urdf/eve_kia_soul_ev.xacro (robot description, xacro)
@@ -18,9 +18,9 @@
   <xacro:include filename="eve_mirror_mount_left.xacro"/>
   <xacro:include filename="eve_mirror_mount_right.xacro"/>
-  <xacro:mirror_mount_left parent="base_link">
-    <origin xyz="0.95 0.88 1.26" rpy="0 0 0"/>
+  <xacro:mirror_mount_left parent="lidar_top">
+    <origin xyz="0.924884 -0.972881 -0.840734" rpy="0.017163 0.108708 -0.580009"/>
   </xacro:mirror_mount_left>
-  <xacro:mirror_mount_right parent="base_link">
-    <origin xyz="0.95 -0.88 1.26" rpy="0 0 0"/>
+  <xacro:mirror_mount_right parent="lidar_top">
+    <origin xyz="1.102008 0.748385 -0.824361" rpy="0.049416 0.068287 0.246267"/>
   </xacro:mirror_mount_right>
 </robot>

Commit message: naming convention and flip

File: src/interfacing/eve_description/urdf/eve_kia_soul_ev.xacro (robot description, xacro)
@@ -16,11 +16,11 @@
   </xacro:roof_mount>
   <!-- Include mirror mounts and sensors -->
-  <xacro:include filename="eve_mirror_mount_left.xacro"/>
-  <xacro:include filename="eve_mirror_mount_right.xacro"/>
-  <xacro:mirror_mount_left parent="lidar_top">
+  <xacro:include filename="eve_mirror_mount_nw.xacro"/>
+  <xacro:include filename="eve_mirror_mount_ne.xacro"/>
+  <xacro:mirror_mount_ne parent="lidar_cc">
     <origin xyz="0.924884 -0.972881 -0.840734" rpy="0.017163 0.108708 -0.580009"/>
-  </xacro:mirror_mount_left>
-  <xacro:mirror_mount_right parent="lidar_top">
+  </xacro:mirror_mount_ne>
+  <xacro:mirror_mount_nw parent="lidar_cc">
     <origin xyz="1.102008 0.748385 -0.824361" rpy="0.049416 0.068287 0.246267"/>
-  </xacro:mirror_mount_right>
+  </xacro:mirror_mount_nw>
 </robot>

File: src/interfacing/eve_description/urdf/eve_mirror_mount_ne.xacro (robot description, xacro)
@@ -2,14 +2,14 @@
 <robot xmlns:xacro="http://ros.org/wiki/xacro">
   <!-- Mirror mount macro - allows parent specification -->
-  <xacro:macro name="mirror_mount_right" params="parent *origin">
+  <xacro:macro name="mirror_mount_nw" params="parent *origin">
     <!-- Mirror mount for all sensors -->
-    <link name="mirror_mount_right"/>
-    <joint name="mirror_mount_right_joint" type="fixed">
+    <link name="mirror_mount_nw"/>
+    <joint name="mirror_mount_nw_joint" type="fixed">
       <parent link="${parent}"/>
-      <child link="mirror_mount_right"/>
+      <child link="mirror_mount_nw"/>
       <xacro:insert_block name="origin"/>
     </joint>
-    <!-- Right LiDAR -->
-    <link name="lidar_NE">
+    <!-- Left LiDAR -->
+    <link name="lidar_nw">
       <visual>
         <origin xyz="0 0 0" rpy="0 0 0"/>
@@ -28,7 +28,7 @@
       </collision>
     </link>
-    <joint name="lidar_NE_mount_yaw" type="fixed">
-      <parent link="mirror_mount_right"/>
-      <child link="lidar_NE"/>
+    <joint name="lidar_nw_mount_yaw" type="fixed">
+      <parent link="mirror_mount_nw"/>
+      <child link="lidar_nw"/>
       <origin xyz="0 0 0" rpy="0 0 0"/>
     </joint>

File: src/interfacing/eve_description/urdf/eve_mirror_mount_nw.xacro (robot description, xacro)
@@ -2,14 +2,14 @@
 <robot xmlns:xacro="http://ros.org/wiki/xacro">
   <!-- Mirror mount macro - allows parent specification -->
-  <xacro:macro name="mirror_mount_left" params="parent *origin">
+  <xacro:macro name="mirror_mount_ne" params="parent *origin">
     <!-- Mirror mount for all sensors -->
-    <link name="mirror_mount_left"/>
-    <joint name="mirror_mount_left_joint" type="fixed">
+    <link name="mirror_mount_ne"/>
+    <joint name="mirror_mount_ne_joint" type="fixed">
       <parent link="${parent}"/>
-      <child link="mirror_mount_left"/>
+      <child link="mirror_mount_ne"/>
       <xacro:insert_block name="origin"/>
     </joint>
-    <!-- Left LiDAR -->
-    <link name="lidar_NW">
+    <!-- Right LiDAR -->
+    <link name="lidar_ne">
       <visual>
         <origin xyz="0 0 0" rpy="0 0 0"/>
@@ -28,7 +28,7 @@
       </collision>
     </link>
-    <joint name="lidar_NW_mount_yaw" type="fixed">
-      <parent link="mirror_mount_left"/>
-      <child link="lidar_NW"/>
+    <joint name="lidar_ne_mount_yaw" type="fixed">
+      <parent link="mirror_mount_ne"/>
+      <child link="lidar_ne"/>
       <origin xyz="0 0 0" rpy="0 0 0"/>
     </joint>

File: src/interfacing/eve_description/urdf/eve_roof_mount.xacro (robot description, xacro)
@@ -11,5 +11,5 @@
     </joint>
     <!-- Top LiDAR -->
-    <link name="lidar_top">
+    <link name="lidar_cc">
       <visual>
         <origin xyz="0 0 0" rpy="0 0 0"/>
@@ -28,7 +28,7 @@
       </collision>
     </link>
-    <joint name="lidar_top_mount_yaw" type="fixed">
+    <joint name="lidar_cc_mount_yaw" type="fixed">
       <parent link="roof_mount"/>
-      <child link="lidar_top"/>
+      <child link="lidar_cc"/>
       <origin xyz="0 0 0.35" rpy="0 0 0"/>
     </joint>

Commit message: enabling auto-exposure and gain settings

File: src/interfacing/eve_description/urdf/eve_kia_soul_ev.xacro (robot description, xacro)
@@ -13,5 +13,5 @@
   <!-- Instantiate roof mount with position relative to chassis -->
   <xacro:roof_mount parent="base_link">
-    <origin xyz="0 0 1.76" rpy="0 0 0"/>
+    <origin xyz="0 0 1.72" rpy="0 0 0"/>
   </xacro:roof_mount>
   <!-- Include mirror mounts and sensors -->

File: src/interfacing/eve_description/urdf/eve_roof_mount.xacro (robot description, xacro)
@@ -31,5 +31,5 @@
       <parent link="roof_mount"/>
       <child link="lidar_cc"/>
-      <origin xyz="0 0 0.35" rpy="0 0 0"/>
+      <origin xyz="0 0 0.35" rpy="0 0 0.10472"/>
     </joint>
     <!-- GPS/IMU Antenna -->

Commit message: lower camera nominal extrinsics

File: src/interfacing/eve_description/urdf/eve_kia_soul_ev.xacro (robot description, xacro)
@@ -15,4 +15,6 @@
     <origin xyz="0 0 1.76" rpy="0 0 0"/>
   </xacro:roof_mount>
+  <!-- Nominal lower camera extrinsics (placeholder values; update once measured) -->
+  <xacro:lower_cameras parent="base_link"/>
   <!-- Include mirror mounts and sensors -->
   <xacro:include filename="eve_mirror_mount_nw.xacro"/>

File: src/interfacing/eve_description/urdf/eve_roof_mount.xacro (robot description, xacro)
@@ -97,3 +97,42 @@
     <xacro:create_camera index="7" name="nn"/>
   </xacro:macro>
+  <!-- Lower cameras (nominal extrinsics; update xyz/rpy once measured) -->
+  <xacro:macro name="lower_cameras" params="parent">
+    <!--
+      Convention: camera link is used directly as frame_id (no separate optical frame).
+      The additional roll of -pi/2 follows the pano camera convention to go from FLU to RDF.
+    -->
+    <xacro:property name="low_cam_x" value="1.50"/>
+    <xacro:property name="low_cam_y" value="0.85"/>
+    <xacro:property name="low_cam_z" value="0.75"/>
+    <!-- Cardinal-ish yaws for nominal mounting directions -->
+    <xacro:property name="yaw_ne" value="${pi/4}"/>
+    <xacro:property name="yaw_se" value="${-pi/4}"/>
+    <xacro:property name="yaw_sw" value="${-3*pi/4}"/>
+    <xacro:property name="yaw_nw" value="${3*pi/4}"/>
+    <link name="camera_low_ne"/>
+    <joint name="camera_low_ne_mount" type="fixed">
+      <parent link="${parent}"/>
+      <child link="camera_low_ne"/>
+      <origin xyz="${low_cam_x} ${-low_cam_y} ${low_cam_z}" rpy="${-pi/2} 0 ${yaw_ne - pi/2}"/>
+    </joint>
+    <link name="camera_low_se"/>
+    <joint name="camera_low_se_mount" type="fixed">
+      <parent link="${parent}"/>
+      <child link="camera_low_se"/>
+      <origin xyz="${low_cam_x} ${-low_cam_y} ${low_cam_z}" rpy="${-pi/2} 0 ${yaw_se - pi/2}"/>
+    </joint>
+    <link name="camera_low_sw"/>
+    <joint name="camera_low_sw_mount" type="fixed">
+      <parent link="${parent}"/>
+      <child link="camera_low_sw"/>
+      <origin xyz="${-low_cam_x} ${-low_cam_y} ${low_cam_z}" rpy="${-pi/2} 0 ${yaw_sw - pi/2}"/>
+    </joint>
+    <link name="camera_low_nw"/>
+    <joint name="camera_low_nw_mount" type="fixed">
+      <parent link="${parent}"/>
+      <child link="camera_low_nw"/>
+      <origin xyz="${-low_cam_x} ${low_cam_y} ${low_cam_z}" rpy="${-pi/2} 0 ${yaw_nw - pi/2}"/>
+    </joint>
+  </xacro:macro>
 </robot>

Commit message: rename roof_mount to base_link, remove old base link

File: src/interfacing/eve_description/urdf/eve_kia_soul_ev.xacro (robot description, xacro)
@@ -7,14 +7,12 @@
   <!-- Instantiate chassis with position relative to base_link -->
   <xacro:chassis parent="base_link">
-    <origin xyz="-0.8629 0 0" rpy="0 0 0"/>
+    <origin xyz="-0.8629 0 -1.76" rpy="0 0 0"/>
   </xacro:chassis>
   <!-- Include roof mount and sensors -->
   <xacro:include filename="eve_roof_mount.xacro"/>
-  <!-- Instantiate roof mount with position relative to chassis -->
-  <xacro:roof_mount parent="base_link">
-    <origin xyz="0 0 1.76" rpy="0 0 0"/>
-  </xacro:roof_mount>
+  <!-- Base link is the roof frame; attach roof sensors directly to base_link -->
+  <xacro:roof_mount parent="base_link"/>
   <!-- Nominal lower camera extrinsics (placeholder values; update once measured) -->
-  <xacro:lower_cameras parent="roof_mount"/>
+  <xacro:lower_cameras parent="base_link"/>
   <!-- Include mirror mounts and sensors -->
   <xacro:include filename="eve_mirror_mount_nw.xacro"/>

File: src/interfacing/eve_description/urdf/eve_roof_mount.xacro (robot description, xacro)
@@ -1,13 +1,6 @@
 <?xml version="1.0"?>
 <robot xmlns:xacro="http://ros.org/wiki/xacro">
-  <!-- Roof mount macro - allows parent specification -->
-  <xacro:macro name="roof_mount" params="parent *origin">
-    <!-- Roof mount for all sensors -->
-    <link name="roof_mount"/>
-    <joint name="roof_mount_joint" type="fixed">
-      <parent link="${parent}"/>
-      <child link="roof_mount"/>
-      <xacro:insert_block name="origin"/>
-    </joint>
+  <!-- Roof mount macro - attaches sensors to the provided parent link -->
+  <xacro:macro name="roof_mount" params="parent">
     <!-- Top LiDAR -->
     <link name="lidar_cc">
@@ -29,5 +22,5 @@
     </link>
     <joint name="lidar_cc_mount_yaw" type="fixed">
-      <parent link="roof_mount"/>
+      <parent link="${parent}"/>
       <child link="lidar_cc"/>
       <origin xyz="0 0 0.35" rpy="0 0 0"/>
@@ -52,5 +45,5 @@
     </link>
     <joint name="gps_imu_mount_yaw" type="fixed">
-      <parent link="roof_mount"/>
+      <parent link="${parent}"/>
       <child link="gps_imu_antenna"/>
       <origin xyz="-0.5600 0 0" rpy="0 0 0"/>
@@ -83,5 +76,5 @@
       <!-- the additional rotation of -pi/2 is to go from FLU to RDF coordinate systems -->
       <joint name="camera_pano_${name}_mount" type="fixed">
-        <parent link="roof_mount"/>
+        <parent link="${parent}"/>
         <child link="camera_pano_${name}"/>
         <origin xyz="${cam_x} ${cam_y} ${camera_z}" rpy="${-pi/2} 0 ${angle - pi/2}"/>
