Commit message: Update nominal extrinsics of lower camera (#300)
Co-authored-by: Matthew0803 <matthewfc83@gmail.com>

File: src/interfacing/eve_description/urdf/eve_kia_soul_ev.xacro (robot description, xacro)
@@ -7,12 +7,10 @@
   <!-- Instantiate chassis with position relative to base_link -->
   <xacro:chassis parent="base_link">
-    <origin xyz="-0.8629 0 0" rpy="0 0 0"/>
+    <origin xyz="-0.8629 0 -1.76" rpy="0 0 0"/>
   </xacro:chassis>
   <!-- Include roof mount and sensors -->
   <xacro:include filename="eve_roof_mount.xacro"/>
-  <!-- Instantiate roof mount with position relative to chassis -->
-  <xacro:roof_mount parent="base_link">
-    <origin xyz="0 0 1.76" rpy="0 0 0"/>
-  </xacro:roof_mount>
+  <!-- Base link is the roof frame; attach roof sensors directly to base_link -->
+  <xacro:roof_mount parent="base_link"/>
   <!-- Nominal lower camera extrinsics (placeholder values; update once measured) -->
   <xacro:lower_cameras parent="base_link"/>

File: src/interfacing/eve_description/urdf/eve_roof_mount.xacro (robot description, xacro)
@@ -1,13 +1,6 @@
 <?xml version="1.0"?>
 <robot xmlns:xacro="http://ros.org/wiki/xacro">
-  <!-- Roof mount macro - allows parent specification -->
-  <xacro:macro name="roof_mount" params="parent *origin">
-    <!-- Roof mount for all sensors -->
-    <link name="roof_mount"/>
-    <joint name="roof_mount_joint" type="fixed">
-      <parent link="${parent}"/>
-      <child link="roof_mount"/>
-      <xacro:insert_block name="origin"/>
-    </joint>
+  <!-- Roof mount macro - attaches sensors to the provided parent link -->
+  <xacro:macro name="roof_mount" params="parent">
     <!-- Top LiDAR -->
     <link name="lidar_cc">
@@ -29,5 +22,5 @@
     </link>
     <joint name="lidar_cc_mount_yaw" type="fixed">
-      <parent link="roof_mount"/>
+      <parent link="${parent}"/>
       <child link="lidar_cc"/>
       <origin xyz="0 0 0.35" rpy="0 0 0"/>
@@ -52,5 +45,5 @@
     </link>
     <joint name="gps_imu_mount_yaw" type="fixed">
-      <parent link="roof_mount"/>
+      <parent link="${parent}"/>
       <child link="gps_imu_antenna"/>
       <origin xyz="-0.5600 0 0" rpy="0 0 0"/>
@@ -83,5 +76,5 @@
       <!-- the additional rotation of -pi/2 is to go from FLU to RDF coordinate systems -->
       <joint name="camera_pano_${name}_mount" type="fixed">
-        <parent link="roof_mount"/>
+        <parent link="${parent}"/>
         <child link="camera_pano_${name}"/>
         <origin xyz="${cam_x} ${cam_y} ${camera_z}" rpy="${-pi/2} 0 ${angle - pi/2}"/>
@@ -99,17 +92,18 @@
   <!-- Lower cameras (nominal extrinsics; update xyz/rpy once measured) -->
   <xacro:macro name="lower_cameras" params="parent">
-    <xacro:property name="low_cam_x" value="1.50"/>
-    <xacro:property name="low_cam_y" value="0.85"/>
-    <xacro:property name="low_cam_z" value="0.75"/>
+    <xacro:property name="low_cam_x_forward" value="0.6125"/>
+    <xacro:property name="low_cam_x_backward" value="0.775"/>
+    <xacro:property name="low_cam_y" value="0.725"/>
+    <xacro:property name="low_cam_z" value="0.034"/>
     <!-- Nominal yaws in the vehicle FLU frame (front=+x, left=+y), estimated from sensor_convention -->
-    <xacro:property name="yaw_ne" value="${-5*pi/6}"/>  <!-- ~ -150 deg -->
-    <xacro:property name="yaw_se" value="${-pi/6}"/>    <!-- ~ -30 deg -->
-    <xacro:property name="yaw_sw" value="${pi/6}"/>     <!-- ~ 30 deg -->
-    <xacro:property name="yaw_nw" value="${5*pi/6}"/>   <!-- ~ 150 deg -->
+    <xacro:property name="yaw_ne" value="${-2.4434}"/>  <!-- ~ -150 deg -->
+    <xacro:property name="yaw_se" value="${0.8726}"/>    <!-- ~ -30 deg -->
+    <xacro:property name="yaw_sw" value="${2.4434}"/>     <!-- ~ 30 deg -->
+    <xacro:property name="yaw_nw" value="${-0.8726}"/>   <!-- ~ 150 deg -->
     <link name="camera_lower_ne"/>
     <joint name="camera_lower_ne_mount" type="fixed">
       <parent link="${parent}"/>
       <child link="camera_lower_ne"/>
-      <origin xyz="${low_cam_x} ${-low_cam_y} ${low_cam_z}" rpy="${-pi/2} 0 ${yaw_ne - pi/2}"/>
+      <origin xyz="${low_cam_x_forward} ${-low_cam_y} ${-low_cam_z}" rpy="${-pi/2} 0 ${yaw_ne - pi/2}"/>
     </joint>
     <link name="camera_lower_se"/>
@@ -117,5 +111,5 @@
       <parent link="${parent}"/>
       <child link="camera_lower_se"/>
-      <origin xyz="${-low_cam_x} ${-low_cam_y} ${low_cam_z}" rpy="${-pi/2} 0 ${yaw_se - pi/2}"/>
+      <origin xyz="${-low_cam_x_backward} ${-low_cam_y} ${-low_cam_z}" rpy="${-pi/2} 0 ${yaw_se - pi}"/>
     </joint>
     <link name="camera_lower_sw"/>
@@ -123,5 +117,5 @@
       <parent link="${parent}"/>
       <child link="camera_lower_sw"/>
-      <origin xyz="${-low_cam_x} ${low_cam_y} ${low_cam_z}" rpy="${-pi/2} 0 ${yaw_sw - pi/2}"/>
+      <origin xyz="${-low_cam_x_backward} ${low_cam_y} ${-low_cam_z}" rpy="${-pi/2} 0 ${yaw_sw - pi}"/>
     </joint>
     <link name="camera_lower_nw"/>
@@ -129,5 +123,5 @@
       <parent link="${parent}"/>
       <child link="camera_lower_nw"/>
-      <origin xyz="${low_cam_x} ${low_cam_y} ${low_cam_z}" rpy="${-pi/2} 0 ${yaw_nw - pi/2}"/>
+      <origin xyz="${low_cam_x_forward} ${low_cam_y} ${-low_cam_z}" rpy="${-pi/2} 0 ${yaw_nw + pi/2}"/>
     </joint>
   </xacro:macro>

Commit message: Under Revertion of Sensor Tuning (#342)
* Update watod-config.sh

* enabling auto-exposure and gain settings

* enabling auto-exposure and gain settings (#288)

* accept this imperfect world

File: src/interfacing/eve_description/urdf/eve_kia_soul_ev.xacro (robot description, xacro)
@@ -7,5 +7,5 @@
   <!-- Instantiate chassis with position relative to base_link -->
   <xacro:chassis parent="base_link">
-    <origin xyz="-0.8629 0 -1.76" rpy="0 0 0"/>
+    <origin xyz="-0.8629 0 -1.72" rpy="0 0 0"/>
   </xacro:chassis>
   <!-- Include roof mount and sensors -->

File: src/interfacing/eve_description/urdf/eve_roof_mount.xacro (robot description, xacro)
@@ -24,5 +24,5 @@
       <parent link="${parent}"/>
       <child link="lidar_cc"/>
-      <origin xyz="0 0 0.35" rpy="0 0 0"/>
+      <origin xyz="0 0 0.35" rpy="0 0 0.10472"/>
     </joint>
     <!-- GPS/IMU Antenna -->

Commit message: base_link to base_footprint

File: src/interfacing/eve_description/urdf/eve_kia_soul_ev.xacro (robot description, xacro)
@@ -1,6 +1,13 @@
 <?xml version="1.0"?>
 <robot name="eve_kia_soul_ev" xmlns:xacro="http://ros.org/wiki/xacro">
-  <!-- Base link (root of the robot) -->
+  <!-- Base footprint (root of the robot, on the ground plane) -->
+  <link name="base_footprint"/>
+  <!-- Base link (roof frame, 1.76m above ground) -->
   <link name="base_link"/>
+  <joint name="base_footprint_joint" type="fixed">
+    <parent link="base_footprint"/>
+    <child link="base_link"/>
+    <origin xyz="0 0 1.76" rpy="0 0 0"/>
+  </joint>
   <!-- Include chassis -->
   <xacro:include filename="eve_chassis.xacro"/>

Commit message: adjust lidar extrinsics

File: src/interfacing/eve_description/urdf/eve_kia_soul_ev.xacro (robot description, xacro)
@@ -26,8 +26,8 @@
   <xacro:include filename="eve_mirror_mount_ne.xacro"/>
   <xacro:mirror_mount_ne parent="lidar_cc">
-    <origin xyz="0.924884 -0.972881 -0.840734" rpy="0.017163 0.108708 -0.580009"/>
+    <origin xyz="0.940111 -0.949479 -0.841508" rpy="0.025541 0.108090 -0.583396"/>
   </xacro:mirror_mount_ne>
   <xacro:mirror_mount_nw parent="lidar_cc">
-    <origin xyz="1.102008 0.748385 -0.824361" rpy="0.049416 0.068287 0.246267"/>
+    <origin xyz="1.074790 0.806157 -0.816995" rpy="0.049541 0.067085 0.244440"/>
   </xacro:mirror_mount_nw>
 </robot>

Commit message: weird issues with quarternion -> euler rotation conversion, fixed

File: src/interfacing/eve_description/urdf/eve_kia_soul_ev.xacro (robot description, xacro)
@@ -26,8 +26,8 @@
   <xacro:include filename="eve_mirror_mount_ne.xacro"/>
   <xacro:mirror_mount_ne parent="lidar_cc">
-    <origin xyz="0.940111 -0.949479 -0.841508" rpy="0.025541 0.108090 -0.583396"/>
+    <origin xyz="0.944015 -0.939612 -0.842884" rpy="-0.038481 0.104171 -0.584697"/>
   </xacro:mirror_mount_ne>
   <xacro:mirror_mount_nw parent="lidar_cc">
-    <origin xyz="1.074790 0.806157 -0.816995" rpy="0.049541 0.067085 0.244440"/>
+    <origin xyz="1.072228 0.817496 -0.820133" rpy="0.064777 0.052500 0.247888"/>
   </xacro:mirror_mount_nw>
 </robot>

Commit message: adding initial est of imu to lidar

File: src/interfacing/eve_description/urdf/eve_kia_soul_ev.xacro (robot description, xacro)
@@ -1,23 +1,19 @@
 <?xml version="1.0"?>
 <robot name="eve_kia_soul_ev" xmlns:xacro="http://ros.org/wiki/xacro">
-  <!-- Base footprint (root of the robot, on the ground plane) -->
-  <link name="base_footprint"/>
-  <!-- Base link (roof frame, 1.76m above ground) -->
+  <!-- Base link (root of the robot) -->
   <link name="base_link"/>
-  <joint name="base_footprint_joint" type="fixed">
-    <parent link="base_footprint"/>
-    <child link="base_link"/>
-    <origin xyz="0 0 1.76" rpy="0 0 0"/>
-  </joint>
   <!-- Include chassis -->
   <xacro:include filename="eve_chassis.xacro"/>
   <!-- Instantiate chassis with position relative to base_link -->
   <xacro:chassis parent="base_link">
-    <origin xyz="-0.8629 0 -1.72" rpy="0 0 0"/>
+    <origin xyz="-0.8629 0 -1.76" rpy="0 0 0"/>
   </xacro:chassis>
   <!-- Include roof mount and sensors -->
   <xacro:include filename="eve_roof_mount.xacro"/>
   <!-- Base link is the roof frame; attach roof sensors directly to base_link -->
-  <xacro:roof_mount parent="base_link"/>
+  <xacro:roof_mount
+    parent="base_link"
+    imu_xyz="-0.4090656 0.3916093 -0.1823015"
+    imu_rpy="-0.01013236 0.00230282 -0.81890701"/>
   <!-- Nominal lower camera extrinsics (placeholder values; update once measured) -->
   <xacro:lower_cameras parent="base_link"/>
@@ -26,8 +22,8 @@
   <xacro:include filename="eve_mirror_mount_ne.xacro"/>
   <xacro:mirror_mount_ne parent="lidar_cc">
-    <origin xyz="0.944015 -0.939612 -0.842884" rpy="-0.038481 0.104171 -0.584697"/>
+    <origin xyz="0.924884 -0.972881 -0.840734" rpy="0.017163 0.108708 -0.580009"/>
   </xacro:mirror_mount_ne>
   <xacro:mirror_mount_nw parent="lidar_cc">
-    <origin xyz="1.072228 0.817496 -0.820133" rpy="0.064777 0.052500 0.247888"/>
+    <origin xyz="1.102008 0.748385 -0.824361" rpy="0.049416 0.068287 0.246267"/>
   </xacro:mirror_mount_nw>
 </robot>

File: src/interfacing/eve_description/urdf/eve_roof_mount.xacro (robot description, xacro)
@@ -2,5 +2,5 @@
 <robot xmlns:xacro="http://ros.org/wiki/xacro">
   <!-- Roof mount macro - attaches sensors to the provided parent link -->
-  <xacro:macro name="roof_mount" params="parent">
+  <xacro:macro name="roof_mount" params="parent imu_xyz:='-0.5600 0 0' imu_rpy:='0 0 0'">
     <!-- Top LiDAR -->
     <link name="lidar_cc">
@@ -24,5 +24,12 @@
       <parent link="${parent}"/>
       <child link="lidar_cc"/>
-      <origin xyz="0 0 0.35" rpy="0 0 0.10472"/>
+      <origin xyz="0 0 0.35" rpy="0 0 0"/>
+    </joint>
+    <!-- Alias frame to match bag/driver frame_id (lidar_top) -->
+    <link name="lidar_top"/>
+    <joint name="lidar_top_alias" type="fixed">
+      <parent link="lidar_cc"/>
+      <child link="lidar_top"/>
+      <origin xyz="0 0 0" rpy="0 0 0"/>
     </joint>
     <!-- GPS/IMU Antenna -->
@@ -48,4 +55,26 @@
       <child link="gps_imu_antenna"/>
       <origin xyz="-0.5600 0 0" rpy="0 0 0"/>
+    </joint>
+    <link name="imu_link">
+      <visual>
+        <origin xyz="0 0 0" rpy="0 0 0"/>
+        <geometry>
+          <sphere radius="0.04"/>
+        </geometry>
+        <material name="green">
+          <color rgba="0.0 1.0 0.0 1"/>
+        </material>
+      </visual>
+      <collision>
+        <origin xyz="0 0 0" rpy="0 0 0"/>
+        <geometry>
+          <sphere radius="0.04"/>
+        </geometry>
+      </collision>
+    </link>
+    <joint name="imu_mount" type="fixed">
+      <parent link="${parent}"/>
+      <child link="imu_link"/>
+      <origin xyz="${imu_xyz}" rpy="${imu_rpy}"/>
     </joint>
     <xacro:property name="camera_z" value="0.217"/>

Commit message: working imu integration factor

File: src/interfacing/eve_description/urdf/eve_kia_soul_ev.xacro (robot description, xacro)
@@ -1,11 +1,19 @@
 <?xml version="1.0"?>
 <robot name="eve_kia_soul_ev" xmlns:xacro="http://ros.org/wiki/xacro">
-  <!-- Base link (root of the robot) -->
+  <!-- Base footprint (root of the robot, on the ground plane) -->
+  <link name="base_footprint"/>
+  <!-- Base link (roof frame, 1.76m above ground) -->
   <link name="base_link"/>
+  <joint name="base_footprint_joint" type="fixed">
+    <parent link="base_footprint"/>
+    <child link="base_link"/>
+    <origin xyz="0 0 1.76" rpy="0 0 0"/>
+  </joint>
   <!-- Include chassis -->
   <xacro:include filename="eve_chassis.xacro"/>
-  <!-- Instantiate chassis with position relative to base_link -->
-  <xacro:chassis parent="base_link">
-    <origin xyz="-0.8629 0 -1.76" rpy="0 0 0"/>
+  <!-- Instantiate chassis with position relative to base_footprint -->
+  <!-- x: rear axle is 0.8629m behind sensor mast -->
+  <xacro:chassis parent="base_footprint">
+    <origin xyz="-0.8629 0 0" rpy="0 0 0"/>
   </xacro:chassis>
   <!-- Include roof mount and sensors -->
@@ -15,5 +23,5 @@
     parent="base_link"
     imu_xyz="-0.973762 -0.033626 -1.316802"
-    imu_rpy="-0.006167 0.042198 -1.653916"/>
+    imu_rpy="-0.006167 0.042198 -0.083116"/>
   <!-- Nominal lower camera extrinsics (placeholder values; update once measured) -->
   <xacro:lower_cameras parent="base_link"/>
@@ -22,8 +30,8 @@
   <xacro:include filename="eve_mirror_mount_ne.xacro"/>
   <xacro:mirror_mount_ne parent="lidar_cc">
-    <origin xyz="0.924884 -0.972881 -0.840734" rpy="0.017163 0.108708 -0.580009"/>
+    <origin xyz="0.944015 -0.939612 -0.842884" rpy="-0.038481 0.104171 -0.584697"/>
   </xacro:mirror_mount_ne>
   <xacro:mirror_mount_nw parent="lidar_cc">
-    <origin xyz="1.102008 0.748385 -0.824361" rpy="0.049416 0.068287 0.246267"/>
+    <origin xyz="1.072228 0.817496 -0.820133" rpy="0.064777 0.052500 0.247888"/>
   </xacro:mirror_mount_nw>
 </robot>

File: src/interfacing/eve_description/urdf/eve_roof_mount.xacro (robot description, xacro)
@@ -24,5 +24,5 @@
       <parent link="${parent}"/>
       <child link="lidar_cc"/>
-      <origin xyz="0 0 0.35" rpy="0 0 0"/>
+      <origin xyz="0 0 0.35" rpy="0 0 0.10472"/>
     </joint>
     <!-- Alias frame to match bag/driver frame_id (lidar_top) -->
@@ -74,5 +74,5 @@
     </link>
     <joint name="imu_mount" type="fixed">
-      <parent link="${parent}"/>
+      <parent link="lidar_cc"/>
       <child link="imu_link"/>
       <origin xyz="${imu_xyz}" rpy="${imu_rpy}"/>

Commit message: added package for lidar imu calibration (#376)
* added package for lidar imu calibration

* cleanup

* pre-commit

File: src/interfacing/eve_description/urdf/eve_kia_soul_ev.xacro (robot description, xacro)
@@ -20,5 +20,8 @@
   <xacro:include filename="eve_roof_mount.xacro"/>
   <!-- Base link is the roof frame; attach roof sensors directly to base_link -->
-  <xacro:roof_mount parent="base_link"/>
+  <xacro:roof_mount
+    parent="base_link"
+    imu_xyz="-0.973762 -0.033626 -1.316802"
+    imu_rpy="-0.006167 0.042198 -0.083116"/>
   <!-- Nominal lower camera extrinsics (placeholder values; update once measured) -->
   <xacro:lower_cameras parent="base_link"/>

File: src/interfacing/eve_description/urdf/eve_roof_mount.xacro (robot description, xacro)
@@ -2,5 +2,5 @@
 <robot xmlns:xacro="http://ros.org/wiki/xacro">
   <!-- Roof mount macro - attaches sensors to the provided parent link -->
-  <xacro:macro name="roof_mount" params="parent">
+  <xacro:macro name="roof_mount" params="parent imu_xyz:='-0.5600 0 0' imu_rpy:='0 0 0'">
     <!-- Top LiDAR -->
     <link name="lidar_cc">
@@ -48,4 +48,26 @@
       <child link="gps_imu_antenna"/>
       <origin xyz="-0.5600 0 0" rpy="0 0 0"/>
+    </joint>
+    <link name="imu_link">
+      <visual>
+        <origin xyz="0 0 0" rpy="0 0 0"/>
+        <geometry>
+          <sphere radius="0.04"/>
+        </geometry>
+        <material name="green">
+          <color rgba="0.0 1.0 0.0 1"/>
+        </material>
+      </visual>
+      <collision>
+        <origin xyz="0 0 0" rpy="0 0 0"/>
+        <geometry>
+          <sphere radius="0.04"/>
+        </geometry>
+      </collision>
+    </link>
+    <joint name="imu_mount" type="fixed">
+      <parent link="lidar_cc"/>
+      <child link="imu_link"/>
+      <origin xyz="${imu_xyz}" rpy="${imu_rpy}"/>
     </joint>
     <xacro:property name="camera_z" value="0.217"/>

Commit message: caching changes

File: src/interfacing/eve_description/urdf/eve_kia_soul_ev.xacro (robot description, xacro)
@@ -23,5 +23,5 @@
     parent="base_link"
     imu_xyz="-0.973762 -0.033626 -1.316802"
-    imu_rpy="-0.006167 0.042198 -0.083116"/>
+    imu_rpy="0 0 -0.083116"/>
   <!-- Nominal lower camera extrinsics (placeholder values; update once measured) -->
   <xacro:lower_cameras parent="base_link"/>

File: src/interfacing/eve_description/urdf/eve_roof_mount.xacro (robot description, xacro)
@@ -21,8 +21,14 @@
       </collision>
     </link>
+    <!-- To level the lidar with the ground plane, take the roll and pitch from
+         the calibrated imu_rpy (IMU rotation relative to lidar) and apply them
+         here. Since the IMU is gravity-calibrated, its roll/pitch relative to
+         the lidar reveals the lidar's physical tilt. Absorbing those angles
+         into this joint levels the lidar frame, then zero out the roll/pitch
+         in imu_rpy (in eve_kia_soul_ev.xacro) so the net transform is unchanged. -->
     <joint name="lidar_cc_mount_yaw" type="fixed">
       <parent link="${parent}"/>
       <child link="lidar_cc"/>
-      <origin xyz="0 0 0.35" rpy="0 0 0.10472"/>
+      <origin xyz="0 0 0.35" rpy="-0.006167 0.042198 0.10472"/>
     </joint>
     <!-- Alias frame to match bag/driver frame_id (lidar_top) -->

Commit message: tracking future path and lidar calib

File: src/interfacing/eve_description/urdf/eve_kia_soul_ev.xacro (robot description, xacro)
@@ -30,8 +30,8 @@
   <xacro:include filename="eve_mirror_mount_ne.xacro"/>
   <xacro:mirror_mount_ne parent="lidar_cc">
-    <origin xyz="0.944015 -0.939612 -0.842884" rpy="-0.038481 0.104171 -0.584697"/>
+    <origin xyz="0.908761 -0.968273 -0.833631" rpy="-0.035597 0.105555 -0.609900"/>
   </xacro:mirror_mount_ne>
   <xacro:mirror_mount_nw parent="lidar_cc">
-    <origin xyz="1.072228 0.817496 -0.820133" rpy="0.064777 0.052500 0.247888"/>
+    <origin xyz="1.096882 0.786605 -0.826910" rpy="0.064322 0.051951 0.221166"/>
   </xacro:mirror_mount_nw>
 </robot>
